File: controller_mb_atu.kicad_pcb (KiCad board)
At the start: 2 copper layers, 115 x 69.8 mm, 50 parts, among them J1 AVR-ISP-6, J2 Front panel, J3 CAN, J4 Mini-DIN-6, U1 LM78M05, U2 MCP2551-I-SN, U3 ATmega32M1-AU, U4 ILD20*, U5 ILD20*, U6 ILD20*, U7 TC7662A, U8 LM337, Y1 12MHz

Commit message: Add production files
Other:
- board text added: "H9 controller main board with an ATU interface v0.1 by SQ8KFH"
- board text removed: "H9 controller main board with ATU interface v0.1 by SQ8KFH"
Changed lines of the file:
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@@
   (page A4)
   (title_block
-    (title "H9 controller main board with ATU interface")
+    (title "H9 controller main board with an ATU interface")
     (date 2020-12-23)
     (rev 0.1)
@@
   (gr_line (start 102.5 58) (end 102.5 55.2) (layer Edge.Cuts) (width 0.05))
   (gr_line (start 100 58) (end 102.5 58) (layer Edge.Cuts) (width 0.05))
-  (gr_text "H9 controller main board\nwith ATU interface v0.1\nby SQ8KFH" (at 197.79 116.364) (layer F.SilkS)
+  (gr_text "H9 controller main board\nwith an ATU interface v0.1\nby SQ8KFH" (at 197.79 116.364) (layer F.SilkS)
     (effects (font (size 1.5 1.5) (thickness 0.2)))
   )
@@
   (segment (start 163.5 85.63) (end 159.69 89.44) (width 0.3048) (layer F.Cu) (net 6) (status 10))
   (segment (start 159.69 89.44) (end 159.69 95.5725) (width 0.3048) (layer F.Cu) (net 6))
-  (via (at 155.245 98.33) (size 0.8) (drill 0.4) (layers F.Cu B.Cu) (net 56))
-  (segment (start 153.105 100.47) (end 155.245 98.33) (width 0.3048) (layer F.Cu) (net 56))
-  (segment (start 148.455 100.47) (end 153.105 100.47) (width 0.3048) (layer F.Cu) (net 56) (status 10))
-  (segment (start 155.515222 98.33) (end 156.987012 96.85821) (width 0.3048) (layer B.Cu) (net 56))
-  (via (at 156.987012 96.85821) (size 0.8) (drill 0.4) (layers F.Cu B.Cu) (net 56))
-  (segment (start 155.245 98.33) (end 155.515222 98.33) (width 0.3048) (layer B.Cu) (net 56))
-  (segment (start 158.42 94.2848) (end 158.42 85.63) (width 0.3048) (layer F.Cu) (net 40) (status 20))
-  (segment (start 156.0848 96.62) (end 158.42 94.2848) (width 0.3048) (layer F.Cu) (net 40))
-  (segment (start 155.505 96.62) (end 156.0848 96.62) (width 0.3048) (layer F.Cu) (net 40) (status 10))
   (segment (start 165.005 100.47) (end 177.82 113.285) (width 0.3048) (layer F.Cu) (net 7))
   (segment (start 177.82 113.285) (end 177.82 114.5) (width 0.3048) (layer F.Cu) (net 7) (status 20))
@@
   (segment (start 198.0075 100.87) (end 195.25 100.87) (width 0.3048) (layer F.Cu) (net 33))
   (segment (start 200.33 103.1925) (end 198.0075 100.87) (width 0.3048) (layer F.Cu) (net 33))
-  (segment (start 139.0825 99.67) (end 137.465 101.2875) (width 0.3048) (layer F.Cu) (net 47) (status 20))
-  (segment (start 142.545 99.74) (end 142.615 99.67) (width 0.3048) (layer F.Cu) (net 47))
-  (segment (start 142.545 101.759) (end 142.545 99.74) (width 0.3048) (layer F.Cu) (net 47) (status 10))
-  (segment (start 142.615 99.67) (end 139.0825 99.67) (width 0.3048) (layer F.Cu) (net 47))
-  (segment (start 148.455 99.67) (end 142.615 99.67) (width 0.3048) (layer F.Cu) (net 47) (status 10))
-  (segment (start 139.0575 98.87) (end 137.465 97.2775) (width 0.3048) (layer F.Cu) (net 48) (status 20))
-  (segment (start 142.545 98.775) (end 142.45 98.87) (width 0.3048) (layer F.Cu) (net 48))
-  (segment (start 142.545 96.879) (end 142.545 98.775) (width 0.3048) (layer F.Cu) (net 48) (status 10))
-  (segment (start 142.45 98.87) (end 139.0575 98.87) (width 0.3048) (layer F.Cu) (net 48))
-  (segment (start 148.455 98.87) (end 142.45 98.87) (width 0.3048) (layer F.Cu) (net 48) (status 10))
   (segment (start 156.9614 98.0636) (end 156.955 98.07) (width 0.3048) (layer F.Cu) (net 34) (status 30))
   (via (at 162.865 96.425) (size 0.8) (drill 0.4) (layers F.Cu B.Cu) (net 34))
@@
   (segment (start 200.1125 64.55162) (end 201.783119 62.881001) (width 0.3048) (layer F.Cu) (net 39))
   (segment (start 200.1125 69.12) (end 200.1125 64.55162) (width 0.3048) (layer F.Cu) (net 39) (status 10))
+  (segment (start 158.42 94.2848) (end 158.42 85.63) (width 0.3048) (layer F.Cu) (net 40) (status 20))
+  (segment (start 156.0848 96.62) (end 158.42 94.2848) (width 0.3048) (layer F.Cu) (net 40))
+  (segment (start 155.505 96.62) (end 156.0848 96.62) (width 0.3048) (layer F.Cu) (net 40) (status 10))
   (segment (start 170.342386 79.28) (end 171.755 77.867386) (width 0.3048) (layer F.Cu) (net 40))
   (segment (start 165.46799 79.28) (end 170.342386 79.28) (width 0.3048) (layer F.Cu) (net 40))
@@
   (segment (start 173.8775 73.565) (end 173.2425 74.2) (width 0.3048) (layer F.Cu) (net 46) (status 30))
   (segment (start 180.075 73.565) (end 173.8775 73.565) (width 0.3048) (layer F.Cu) (net 46) (status 30))
+  (segment (start 139.0825 99.67) (end 137.465 101.2875) (width 0.3048) (layer F.Cu) (net 47) (status 20))
+  (segment (start 142.545 99.74) (end 142.615 99.67) (width 0.3048) (layer F.Cu) (net 47))
+  (segment (start 142.545 101.759) (end 142.545 99.74) (width 0.3048) (layer F.Cu) (net 47) (status 10))
+  (segment (start 142.615 99.67) (end 139.0825 99.67) (width 0.3048) (layer F.Cu) (net 47))
+  (segment (start 148.455 99.67) (end 142.615 99.67) (width 0.3048) (layer F.Cu) (net 47) (status 10))
+  (segment (start 139.0575 98.87) (end 137.465 97.2775) (width 0.3048) (layer F.Cu) (net 48) (status 20))
+  (segment (start 142.545 98.775) (end 142.45 98.87) (width 0.3048) (layer F.Cu) (net 48))
+  (segment (start 142.545 96.879) (end 142.545 98.775) (width 0.3048) (layer F.Cu) (net 48) (status 10))
+  (segment (start 142.45 98.87) (end 139.0575 98.87) (width 0.3048) (layer F.Cu) (net 48))
+  (segment (start 148.455 98.87) (end 142.45 98.87) (width 0.3048) (layer F.Cu) (net 48) (status 10))
   (segment (start 198.35 83.69) (end 199.695 85.035) (width 0.3048) (layer F.Cu) (net 49) (status 20))
   (segment (start 193.98 83.69) (end 198.35 83.69) (width 0.3048) (layer F.Cu) (net 49) (status 10))
@@
   (segment (start 154.705 95.695) (end 157.785 92.615) (width 0.3048) (layer F.Cu) (net 55))
   (segment (start 154.705 96.62) (end 154.705 95.695) (width 0.3048) (layer F.Cu) (net 55) (status 10))
+  (via (at 155.245 98.33) (size 0.8) (drill 0.4) (layers F.Cu B.Cu) (net 56))
+  (segment (start 153.105 100.47) (end 155.245 98.33) (width 0.3048) (layer F.Cu) (net 56))
+  (segment (start 148.455 100.47) (end 153.105 100.47) (width 0.3048) (layer F.Cu) (net 56) (status 10))
+  (segment (start 155.515222 98.33) (end 156.987012 96.85821) (width 0.3048) (layer B.Cu) (net 56))
+  (via (at 156.987012 96.85821) (size 0.8) (drill 0.4) (layers F.Cu B.Cu) (net 56))
+  (segment (start 155.245 98.33) (end 155.515222 98.33) (width 0.3048) (layer B.Cu) (net 56))
   (segment (start 159.055 87.535) (end 160.96 85.63) (width 0.3048) (layer F.Cu) (net 56) (status 20))
   (segment (start 159.055 94.790222) (end 159.055 87.535) (width 0.3048) (layer F.Cu) (net 56))

Commit message: v0.2
Parts:
- removed the C13 at (199.7, 87.5)
- removed D4: 4148, Diode_SMD:D_MiniMELF
- removed the R10 at (187.0, 80.5)
- removed the R9 at (202.9, 81.2)
- added BZ1: Buzzer, Buzzer_Beeper:Buzzer_12x9.5RM7.6, F.Cu at (113.3, 106.0)
- added C17: 1uF, Capacitor_SMD:C_1206_3216Metric_Pad1.42x1.75mm_HandSolder, F.Cu at (190.2, 79.9)
- added C7: 47pF, Capacitor_SMD:C_1206_3216Metric_Pad1.42x1.75mm_HandSolder, F.Cu at (135.6, 85.6)
- added C9: 47pF, Capacitor_SMD:C_1206_3216Metric_Pad1.42x1.75mm_HandSolder, F.Cu at (135.6, 78.0)
- added Q1: 2N7002, Package_TO_SOT_SMD:SOT-23, F.Cu at (196.8, 109.2)
- added Q2: 2N7002, Package_TO_SOT_SMD:SOT-23, F.Cu at (196.8, 102.9)
- added Q3: BC817, Package_TO_SOT_SMD:SOT-23, F.Cu at (122.9, 112.3)
- added R2: 1k 0.25W, Resistor_SMD:R_1206_3216Metric_Pad1.42x1.75mm_HandSolder, F.Cu at (190.2, 110.4)
- added R3: 1k 0,25W, Resistor_SMD:R_1206_3216Metric_Pad1.42x1.75mm_HandSolder, F.Cu at (190.2, 106.0)
- added R7: 100k, Resistor_SMD:R_1206_3216Metric_Pad1.42x1.75mm_HandSolder, F.Cu at (205.7, 109.1)
- added R8: 100k, Resistor_SMD:R_1206_3216Metric_Pad1.42x1.75mm_HandSolder, F.Cu at (205.7, 102.9)
- C10: renamed from C9; value 100nF -> 1nF
- C11: renamed from C8; value 100nF -> 1nF
- C14: value 10uF -> 1uF; footprint Capacitor_THT:CP_Radial_D6.3mm_P2.50mm -> Capacitor_SMD:C_1206_3216Metric_Pad1.42x1.75mm_HandSolder
- R13: value 100R -> 680R
- R5: renamed from R6; value 390 -> 10R
- R6: renamed from R2; value 390 -> 10
- RV1: value R_POT -> 10k
- U4, U5: value ILD20* -> ILD213T
- U6: value ILD20* -> TLP185; footprint Package_SO:SOIC-8_3.9x4.9mm_P1.27mm -> Package_SO:SOIC-4_4.55x3.7mm_P2.54mm
- U7: value TC7662A -> TC7662Bx0A; footprint Package_SO:SO-8_3.9x4.9mm_P1.27mm -> Package_SO:SOIC-8_3.9x4.9mm_P1.27mm
- U8: footprint Package_TO_SOT_SMD:SOT-223-3_TabPin2 -> Package_SO:SOIC-8_3.9x4.9mm_P1.27mm
- moved R12 58.7 mm to (121.6, 104.7), turned to 270 degrees
- moved D3 36.4 mm to (200.3, 69.1), turned to 180 degrees
- moved R13 33.2 mm to (192.7, 94.0), turned to 0 degrees
- moved C19 20.3 mm to (186.4, 82.5), turned to 90 degrees
- moved C18 19.6 mm to (190.8, 88.2), turned to 270 degrees
- moved C16 19.4 mm to (200.3, 73.6), turned to 0 degrees
- moved R15 18.9 mm to (186.4, 88.8)
- moved C14 17.7 mm to (203.5, 80.5), turned to 270 degrees
- moved D2 14.4 mm to (125.4, 71.0), turned to 90 degrees
- moved C10 13.0 mm to (201.9, 109.1)
- moved C11 13.0 mm to (201.9, 102.9), turned to 270 degrees
- moved U8 12.5 mm to (197.2, 88.2), turned to 0 degrees
- moved R5 11.7 mm to (190.2, 99.0)
- moved R6 9.17 mm to (202.6, 97.8), turned to 0 degrees
- moved U7 8.13 mm to (197.2, 79.9), turned to 0 degrees
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- renumbered C10 to C12, C11 to C13, C12 to C15, C17 to C16, C15 to C18, C16 to C19, C7 to C8, J3 to J1, J1 to J2, J2 to J3, R7 to R10, R3 to R11, R8 to R14, R11 to R15, R5 to R4, R4 to R9
Connections:
- net /MISO(ALC) renamed /MISO(BUZ)
- net /START renamed /START_TS
- C10 pad 1: Net-(C9-Pad1) -> Net-(C10-Pad1)
- C11 pad 1: Net-(C8-Pad1) -> Net-(C11-Pad1)
- C14 pad 1: Net-(C14-Pad1) -> GNDD
- C15 pad 1: /+13.8V -> Net-(C15-Pad1)
- C16 pad 1: Net-(C17-Pad1) -> Net-(C15-Pad1)
- C18 pad 1: Net-(C15-Pad1) -> Net-(C18-Pad1)
- C19 pad 1: Net-(C15-Pad1) -> Net-(C18-Pad1)
- D3 pad 1: /KEY -> Net-(C15-Pad1)
- D3 pad 2: GNDD -> Net-(D3-Pad2)
- J2 pad 4: /MOSI(ALC_H) -> /MOSI(ALC)
- J4 pad 2: /+13.8V -> Net-(D3-Pad2)
- J4 pad 5: /KEY -> /KEY_TT
- R12 pad 2: Net-(R12-Pad2) -> Net-(Q3-Pad1)
- R13 pad 1: Net-(R13-Pad1) -> GNDD
- R13 pad 2: /ALC -> Net-(R13-Pad2)
- R14 pad 1: Net-(R8-Pad1) -> /MOSI(ALC)
- R14 pad 2: /MOSI(ALC_H) -> Net-(R14-Pad2)
- R15 pad 1: Net-(R10-Pad2) -> Net-(R13-Pad2)
- R15 pad 2: Net-(C15-Pad1) -> Net-(C18-Pad1)
- R5 pad 2: Net-(C9-Pad1) -> Net-(C10-Pad1)
- R6 pad 1: /KEY -> /KEY_TT
- R6 pad 2: Net-(C8-Pad1) -> Net-(C11-Pad1)
- RV1 pad 1: GNDD -> Net-(RV1-Pad1)
- RV1 pad 2: Net-(R13-Pad1) -> /ALC
- RV1 pad 3: Net-(C15-Pad1) -> GNDD
- U3 pad 2: /MOSI(ALC_H) -> /MOSI(ALC)
- U4 pad 1: Net-(C9-Pad1) -> Net-(R2-Pad2)
- U4 pad 2: GNDD -> Net-(Q1-Pad3)
- U4 pad 3: Net-(C8-Pad1) -> Net-(R3-Pad2)
- U4 pad 4: GNDD -> Net-(Q2-Pad3)
- U5 pad 6: /KEY -> /KEY_TT
- U6 pad 1: Net-(R12-Pad2) -> Net-(R14-Pad2)
- U6 pad 3: Net-(R8-Pad1) -> GND
- U6 pad 4: GND -> Net-(C18-Pad1)
- U6 pad 6: GNDD -> Net-(RV1-Pad1)
- U7 pad 1: (no net) -> Net-(C15-Pad1)
- U7 pad 2: Net-(C14-Pad1) -> Net-(C17-Pad1)
- U7 pad 4: Net-(C14-Pad2) -> Net-(C17-Pad2)
- U7 pad 5: Net-(C13-Pad2) -> Net-(C14-Pad2)
- U7 pad 8: Net-(C17-Pad1) -> Net-(C15-Pad1)
- U8 pad 1: Net-(R10-Pad2) -> Net-(C18-Pad1)
- U8 pad 2: Net-(C13-Pad2) -> Net-(C14-Pad2)
- U8 pad 3: Net-(C15-Pad1) -> Net-(C14-Pad2)
Routing:
- net /KEY: track 63.2 -> 0.00 mm
- net /KEY_TT: track 0.00 -> 53.3 mm
- net Net-(C15-Pad1): track 44.7 -> 83.6 mm, vias 0 -> 2
- net /MOSI(ALC_H): track 31.1 -> 0.00 mm
- net /MOSI(ALC): track 0.00 -> 30.2 mm
- net Net-(C13-Pad2): track 27.4 -> 0.00 mm
- net Net-(C10-Pad1): track 0.00 -> 23.8 mm
- net /MISO(BUZ): track 34.0 -> 57.3 mm, vias 0 -> 5
- net Net-(C18-Pad1): track 0.00 -> 22.7 mm
- net /+13.8V: track 20.8 -> 0.00 mm
- net Net-(R10-Pad2): track 19.2 -> 0.00 mm
- net Net-(C9-Pad1): track 18.6 -> 0.00 mm
- net Net-(Q1-Pad3): track 0.00 -> 16.4 mm
- net Net-(R13-Pad2): track 0.00 -> 14.9 mm
- net Net-(C11-Pad1): track 0.00 -> 13.2 mm
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Other:
- board text added: "H9 controller main board with an ATU interface v0.2 by SQ8KFH"
- board text removed: "H9 controller main board with an ATU interface v0.1 by SQ8KFH"

Commit message: Add L1
Parts:
- added L1: DR331-513AE, Filter:Filter_Bourns_SRF0905_6.0x9.2mm, F.Cu at (128.9, 81.9)
- R10, R11, R12, R14: value 390 -> 390R
- R13: value 680R -> 820R
- R6: value 10 -> 10R
- RV1: value 10k -> 20k
- U6: value TLP185 -> TLP185(GR-TPL,E(O
- turned D2 to -90 degrees
Connections:
- C7 pad 2: /CAN_H -> Net-(U2-Pad7)
- C9 pad 1: /CAN_L -> Net-(C9-Pad1)
- J1 pad 1: (no net) -> unconnected-(J1-Pad1)
- J1 pad 4: (no net) -> unconnected-(J1-Pad4)
- J1 pad 6: (no net) -> unconnected-(J1-Pad6)
- J1 pad 8: (no net) -> unconnected-(J1-Pad8)
- J3 pad 19: (no net) -> unconnected-(J3-Pad19)
- U2 pad 5: (no net) -> unconnected-(U2-Pad5)
- U2 pad 6: /CAN_L -> Net-(C9-Pad1)
- U2 pad 7: /CAN_H -> Net-(U2-Pad7)
- U3 pad 21: (no net) -> unconnected-(U3-Pad21)
- U7 pad 6: (no net) -> unconnected-(U7-Pad6)
- U7 pad 7: (no net) -> unconnected-(U7-Pad7)
- U8 pad 5: (no net) -> unconnected-(U8-Pad5)
- U8 pad 8: (no net) -> unconnected-(U8-Pad8)
Routing:
- net Net-(C9-Pad1): track 0.00 -> 16.9 mm
- net /CAN_H: track 34.6 -> 20.0 mm
- net Net-(U2-Pad7): track 0.00 -> 13.9 mm
- net /CAN_L: track 26.5 -> 16.2 mm
- net Net-(R11-Pad1): track 6.61 -> 5.72 mm
- net /MISO(BUZ): track 57.3 -> 56.6 mm
Other:
- net class Default removed
- board text added: "H9 controller main board with an ATU interface v0.3 by SQ8KFH"
- board text removed: "H9 controller main board with an ATU interface v0.2 by SQ8KFH"
